File: hardware/chromapi_motherboard_v1.kicad_pcb (KiCad board)
At the start: 4 copper layers, 143 parts, among them J1 Battery Input, J10 Conn_FSR_TopLeft, J11 Conn_FSR_TopRight, J12 Conn_FSR_BotLeft, J13 Conn_FSR_BotRight, J14 RPI_Connector, J2 Power Switch, J3 USB_C_Receptacle_USB2.0_14P, J4 Conn_ST_STDC14, J5 Conn_TopLeft, J6 Conn_TopRight, J7 Conn_BotLeft, J8 Conn_BotRight, J9 Speaker connector, M1 Noctua NF-A4x10, Q1 PSMN1R5-30YL, Q2 PSMN1R5-30YL, Q3 AO4435, Q4 AO4468, U1 HY2120, U2 CN3302, U3 TPS568230, U4 LD39050PU33R, U5 74AHCT125, U5 SN74AHCT1G125DBVR, U6 STM32G431KBTx, U7 SN74LVC1T45DBV, U8 MAX98357A, U9 BNO055, Y1 32.768k

Commit message: Updating placement
Parts:
- removed the C29 at (143.1, 66.3)
- removed the C37 at (220.5, 33.0)
- removed the C37 at (261.6, 67.1)
- removed the C43 at (35.5, 174.5)
- removed the C43 at (226.5, 30.5)
- removed the C44 at (55.0, 174.5)
- removed the R23 at (266.6, 62.1)
- removed the R24 at (35.5, 160.5)
- removed the R29 at (266.8, 66.6)
- removed the R30 at (35.5, 173.0)
- removed the R31 at (55.0, 173.0)
- removed TP10: TP_FSR_BotLeft, TestPoint:TestPoint_Pad_D1.0mm
- removed TP11: TP_FSR_BotRight, TestPoint:TestPoint_Pad_D1.0mm
- removed TP8: TP_FSR_TopLeft, TestPoint:TestPoint_Pad_D1.0mm
- removed TP9: TP_FSR_TopRight, TestPoint:TestPoint_Pad_D1.0mm
- removed the U5 at (183.7, 17.9)
- removed the U5 at (139.6, 69.3)
- removed the U7 at (111.7, 85.8)
- removed Y1: 32.768k, Crystal:Crystal_SMD_3215-2Pin_3.2x1.5mm
- added C1: 100nF, Capacitor_SMD:C_0603_1608Metric, F.Cu at (41.0, 148.6)
- added C4: 100nF, Capacitor_SMD:C_0603_1608Metric, F.Cu at (35.2, 150.3)
- added C43: 100nF, Capacitor_SMD:C_0603_1608Metric, F.Cu at (111.1, 81.5)
- added R2: 10k, Resistor_SMD:R_0402_1005Metric, F.Cu at (41.5, 143.4)
- added R3: 10k, Resistor_SMD:R_0402_1005Metric, F.Cu at (41.5, 145.4)
- added R32: 10k, Resistor_SMD:R_0402_1005Metric, F.Cu at (47.5, 172.0)
- added R33: 10k, Resistor_SMD:R_0402_1005Metric, F.Cu at (57.0, 172.0)
- added R34: 10k, Resistor_SMD:R_0402_1005Metric, F.Cu at (66.5, 172.0)
- added R35: 10k, Resistor_SMD:R_0402_1005Metric, F.Cu at (75.5, 172.0)
- added R5: 10, Resistor_SMD:R_0603_1608Metric, F.Cu at (41.0, 151.1)
- added R6: 2m, Resistor_SMD:R_2512_6332Metric, F.Cu at (35.6, 144.9)
- added R8: 10, Resistor_SMD:R_0603_1608Metric, F.Cu at (41.0, 153.6)
- added U11: BMI088, Package_LGA:Bosch_LGA-16_4.5x3mm_P0.5mm_LayoutBorder7x1y_ClockwisePinNumbering, F.Cu at (111.0, 84.5)
- added U2: INA226, Package_SO:VSSOP-10_3x3mm_P0.5mm, F.Cu at (35.0, 155.5)
- added U6: SN74LVC1G126DBVR, Chromapi_FP:SOT95P280X145-5N, F.Cu at (153.0, 186.5)
- added U8: SN74LVC1G125DBVR, Chromapi_FP:SOT95P280X145-5N, F.Cu at (153.0, 190.9)
- C38, C41: value 22pF -> 100nF
- C39, C40: footprint Capacitor_SMD:C_0402_1005Metric -> Capacitor_SMD:C_0603_1608Metric
- J10: value Conn_FSR_TopLeft -> Top Left Switch
- J11: value Conn_FSR_TopRight -> Top Right Switch
- J12: value Conn_FSR_BotLeft -> Bottom Left Switch
- J13: value Conn_FSR_BotRight -> Bottom Right Switch
- R26, R27: value 4.7k -> 100; footprint Resistor_SMD:R_0603_1608Metric -> Resistor_SMD:R_0402_1005Metric
- R28: footprint Resistor_SMD:R_0603_1608Metric -> Resistor_SMD:R_0402_1005Metric
- U9: value BNO055 -> SN74AHCT1G125DBVR; footprint Package_LGA:LGA-28_5.2x3.8mm_P0.5mm -> Chromapi_FP:SOT95P280X145-5N
- moved C38 236.3 mm to (46.2, 170.5)
- moved C41 214.3 mm to (74.2, 170.5)
- moved R26 167.1 mm to (157.1, 187.3), turned to 0 degrees
- moved R27 166.7 mm to (157.1, 189.2)
- moved R28 163.3 mm to (157.1, 191.2), turned to 0 degrees
- moved C42 155.6 mm to (112.6, 87.5)
- moved J7 150.5 mm to (92.0, 175.9)
- moved J8 150.5 mm to (104.0, 175.9)
- moved J5 150.3 mm to (92.0, 169.0)
- moved J6 150.2 mm to (104.0, 168.9)
- moved C24 107.0 mm to (148.0, 185.0)
- moved C25 107.0 mm to (152.0, 183.0)
- moved R25 105.3 mm to (157.1, 185.3)
- moved TP5 101.4 mm to (165.5, 182.0)
- moved TP6 97.8 mm to (158.0, 175.5)
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- renumbered C8 to C10, C9 to C11, C10 to C12, C11 to C13, C12 to C14, C13 to C15, C14 to C16, C15 to C17, C16 to C18, C17 to C19, C1 to C2, C18 to C20, C19 to C21, C20 to C22, C21 to C23, C27 to C24, C28 to C25, C22 to C26, C23 to C27, C24 to C28, C25 to C29, C2 to C3, C26 to C30, C30 to C31, C31 to C32, C32 to C33, C33 to C34, C34 to C35, C35 to C36, C36 to C37, C45 to C44, C46 to C45, C3 to C5, C4 to C6, C5 to C7, C6 to C8, C7 to C9, R5 to R10, R6 to R11, R7 to R12, R8 to R13, R9 to R14, R10 to R15, R11 to R16, R12 to R17, R13 to R18, R14 to R19, R15 to R20, R16 to R21, R17 to R22, R18 to R23, R19 to R24, R21 to R29, R20 to R30, R22 to R31, R32 to R36, R2 to R4, R3 to R7, R4 to R9, TP6 to TP5, TP5 to TP6, U8 to U10, U2 to U3, U3 to U4, U4 to U5, U6 to U7
Connections:
- C38 pad 1: Net-(U9-XOUT32) -> /Peripherals (Sensors & Audio)/SW_TopLeft
- C39 pad 1: /Peripherals (Sensors & Audio)/FSR_TopLeft -> /Peripherals (Sensors & Audio)/SW_TopRight
- C40 pad 1: /Peripherals (Sensors & Audio)/FSR_TopRight -> /Peripherals (Sensors & Audio)/SW_BotLeft
- C41 pad 1: Net-(U9-XIN32) -> /Peripherals (Sensors & Audio)/SW_BotRight
- C42 pad 1: Net-(U9-CAP) -> +3.3V
- C7 pad 1: /Power Supply & Charge/V_BATT -> /Power Supply & Charge/V_SYS
- C8 pad 1: /Power Supply & Charge/V_BATT -> /Power Supply & Charge/V_SYS
- C9 pad 1: /Power Supply & Charge/V_BATT -> /Power Supply & Charge/V_SYS
- J10 pad 1: +3.3V -> /Peripherals (Sensors & Audio)/SW_TopLeft
- J10 pad 2: /Peripherals (Sensors & Audio)/FSR_TopLeft -> GND
- J11 pad 1: +3.3V -> /Peripherals (Sensors & Audio)/SW_TopRight
- J11 pad 2: /Peripherals (Sensors & Audio)/FSR_TopRight -> GND
- J12 pad 1: +3.3V -> /Peripherals (Sensors & Audio)/SW_BotLeft
- J12 pad 2: /Peripherals (Sensors & Audio)/FSR_BotLeft -> GND
- J13 pad 1: +3.3V -> /Peripherals (Sensors & Audio)/SW_BotRight
- J13 pad 2: /Peripherals (Sensors & Audio)/FSR_BotRight -> GND
- J14 pad 10: unconnected-(J14-Pin_10-Pad10) -> /Raspberry Pi Interface/UART_RXD
- J14 pad 19: /Raspberry Pi Interface/SPI_MOSI -> unconnected-(J14-Pin_19-Pad19)
- J14 pad 21: /Raspberry Pi Interface/SPI_MISO -> unconnected-(J14-Pin_21-Pad21)
- J14 pad 23: /Raspberry Pi Interface/SPI_SCLK -> unconnected-(J14-Pin_23-Pad23)
- J14 pad 24: /Raspberry Pi Interface/SPI_CS -> unconnected-(J14-Pin_24-Pad24)
- J14 pad 8: unconnected-(J14-Pin_8-Pad8) -> /Raspberry Pi Interface/UART_TXD
- J4 pad 13: /STM32 Microcontroller Core/USART1_RX -> unconnected-(J4-VCP_RX-Pad13)
- J4 pad 14: /STM32 Microcontroller Core/USART1_TX -> unconnected-(J4-VCP_TX-Pad14)
- J5 pad 2: /Power Supply & Charge/V_BATT -> /Power Supply & Charge/V_SYS
- J6 pad 2: /Power Supply & Charge/V_BATT -> /Power Supply & Charge/V_SYS
- J7 pad 2: /Power Supply & Charge/V_BATT -> /Power Supply & Charge/V_SYS
- J8 pad 2: /Power Supply & Charge/V_BATT -> /Power Supply & Charge/V_SYS
- R19 pad 1: /Power Supply & Charge/V_BATT -> /Power Supply & Charge/V_SYS
- R22 pad 2: /Power Supply & Charge/V_BATT -> /Power Supply & Charge/V_SYS
- R25 pad 1: /Peripherals (Sensors & Audio)/FSR_TopRight -> /STM32 Microcontroller Core/SERVO_DATA
- R25 pad 2: GND -> +3.3V
- R26 pad 1: +3.3V -> /STM32 Microcontroller Core/SERVO_DATA
- R26 pad 2: /Peripherals (Sensors & Audio)/IMU_SCL -> Net-(U6-Y)
- R27 pad 1: +3.3V -> Net-(U8-Y)
- R27 pad 2: /Peripherals (Sensors & Audio)/IMU_SDA -> /STM32 Microcontroller Core/USART2_RX
- R28 pad 2: Net-(U9-PS1) -> /STM32 Microcontroller Core/USART2_DE
- R30 pad 2: Net-(U5-Y) -> Net-(U9-Y)
- TP2 pad 1: /Power Supply & Charge/V_BATT -> /Power Supply & Charge/V_SYS
- U4 pad 2: /Power Supply & Charge/V_BATT -> /Power Supply & Charge/V_SYS
- U4 pad 3: /Power Supply & Charge/V_BATT -> /Power Supply & Charge/V_SYS
- U4 pad 4: /Power Supply & Charge/V_BATT -> /Power Supply & Charge/V_SYS
- U4 pad 5: /Power Supply & Charge/V_BATT -> /Power Supply & Charge/V_SYS
- U7 pad 10: /Raspberry Pi Interface/SPI_SCLK -> /Peripherals (Sensors & Audio)/SPI_IMU_SCK
- U7 pad 11: /Raspberry Pi Interface/SPI_MISO -> /Peripherals (Sensors & Audio)/SPI_IMU_MOSI
- U7 pad 12: /Raspberry Pi Interface/SPI_MOSI -> /Peripherals (Sensors & Audio)/SPI_IMU_MISO
- U7 pad 13: /Peripherals (Sensors & Audio)/FSR_TopRight -> /Peripherals (Sensors & Audio)/SPI_CS_ACC
- U7 pad 19: /STM32 Microcontroller Core/USART1_TX -> /Raspberry Pi Interface/UART_RXD
- U7 pad 2: /Peripherals (Sensors & Audio)/FSR_TopLeft -> /Peripherals (Sensors & Audio)/SW_TopLeft
- U7 pad 20: /STM32 Microcontroller Core/USART1_RX -> /Raspberry Pi Interface/UART_TXD
- U7 pad 21: unconnected-(U6-PA11-Pad21) -> /Peripherals (Sensors & Audio)/IMU_INT_ACC
- U7 pad 22: unconnected-(U6-PA12-Pad22) -> /Peripherals (Sensors & Audio)/IMU_INT_GYRO
- U7 pad 25: /Peripherals (Sensors & Audio)/IMU_SDA -> /Power Supply & Charge/I2C_INA_SCL
- U7 pad 27: /Peripherals (Sensors & Audio)/IMU_INT -> /Peripherals (Sensors & Audio)/SW_BotLeft
- U7 pad 28: unconnected-(U6-PB5-Pad28) -> /Peripherals (Sensors & Audio)/SW_BotRight
- U7 pad 29: /STM32 Microcontroller Core/TIM4_CH1 -> /STM32 Microcontroller Core/RGB_LED
- U7 pad 3: /Peripherals (Sensors & Audio)/FSR_BotRight -> /Peripherals (Sensors & Audio)/SW_TopRight
- U7 pad 30: /Peripherals (Sensors & Audio)/IMU_SCL -> /Power Supply & Charge/I2C_INA_SDA
- U7 pad 5: /Peripherals (Sensors & Audio)/FSR_BotLeft -> unconnected-(U7-PA0-Pad5)
- U7 pad 9: /Raspberry Pi Interface/SPI_CS -> /Peripherals (Sensors & Audio)/SPI_CS_GYRO
- U9 pad 1: unconnected-(U9-PIN1-Pad1) -> GND
- U9 pad 2: GND -> /STM32 Microcontroller Core/RGB_LED
- U9 pad 3: +3.3V -> GND
- U9 pad 4: +3.3V -> Net-(U9-Y)
- U9 pad 5: Net-(U9-PS1) -> +5V
