File: hardware/servo_control.kicad_sch (KiCad schematic)
At the start: 4 parts, among them J5 Conn_01x03, J6 Conn_01x03, J7 Conn_01x03, J8 Conn_01x03

Commit message: minor fixes
Parts:
- J5: value Conn_01x03 -> Conn_TopLeft
- J6: value Conn_01x03 -> Conn_TopRight
- J7: value Conn_01x03 -> Conn_BotLeft
- J8: value Conn_01x03 -> Conn_BotRight
Changed lines of the file:
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@@
 			)
 		)
-		(property "Value" "Conn_01x03"
+		(property "Value" "Conn_BotLeft"
 			(at 137.16 110.4899 0)
 			(effects
@@
 			)
 		)
-		(property "Value" "Conn_01x03"
+		(property "Value" "Conn_BotRight"
 			(at 172.72 110.4899 0)
 			(effects
@@
 			)
 		)
-		(property "Value" "Conn_01x03"
+		(property "Value" "Conn_TopRight"
 			(at 172.72 91.4399 0)
 			(effects
@@
 			)
 		)
-		(property "Value" "Conn_01x03"
+		(property "Value" "Conn_TopLeft"
 			(at 137.16 91.4399 0)
 			(effects

Commit message: Updating schematic
Changed lines of the file:
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@@
 					(size 1.27 1.27)
 				)
+				(hide yes)
 			)
 		)
@@
 					(size 1.27 1.27)
 				)
+				(hide yes)
 			)
 		)
@@
 					(size 1.27 1.27)
 				)
+				(hide yes)
 			)
 		)
@@
 					(size 1.27 1.27)
 				)
-			)
-		)
+				(hide yes)
+			)
+		)

Commit message: IMU modification and Power monitor addition
Connections:
- net V_BATT renamed V_SYS
