File: hardware/rpi_interface.kicad_sch (KiCad schematic)
At the start: 5 parts, among them J14 RPI_Connector, M1 Noctua NF-A4x10

Commit message: Updating BOM
Parts:
- C42: value 10µF -> 10uF; symbol Device:C -> Device:C_Polarized
- C43: JLCPCB Part# (none) -> C307331; MPN (none) -> CL05B104KB54PNC
Changed lines of the file:
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@@
 				(font
 					(size 1.27 1.27)
+					(italic yes)
 				)
 			)
 		)
 		(property "MP" ""
+			(at 82.55 116.84 0)
+			(hide yes)
+			(show_name no)
+			(do_not_autoplace no)
+			(effects
+				(font
+					(size 1.27 1.27)
+				)
+			)
+		)
+		(property "MPN" "CL05B104KB54PNC"
+			(at 82.55 116.84 0)
+			(hide yes)
+			(show_name no)
+			(do_not_autoplace no)
+			(effects
+				(font
+					(size 1.27 1.27)
+				)
+			)
+		)
+		(property "JLCPCB Part#" "C307331"
 			(at 82.55 116.84 0)
 			(hide yes)
@@
 	)
 	(symbol
-		(lib_id "Device:C")
+		(lib_id "Device:C_Polarized")
 		(at 71.12 116.84 0)
 		(unit 1)
@@
 		(fields_autoplaced yes)
 		(property "Reference" "C42"
-			(at 74.93 115.5699 0)
+			(at 74.93 114.6809 0)
 			(show_name no)
 			(do_not_autoplace no)
@@
 			)
 		)
-		(property "Value" "10µF"
-			(at 74.93 118.1099 0)
+		(property "Value" "10uF"
+			(at 74.93 117.2209 0)
 			(show_name no)
 			(do_not_autoplace no)
@@
 			)
 		)
-		(property "Description" "Unpolarized capacitor"
+		(property "Description" "Polarized capacitor"
 			(at 71.12 116.84 0)
 			(hide yes)
@@
 			(at 71.12 116.84 0)
 			(hide yes)
+			(show_name no)
+			(do_not_autoplace no)
+			(effects
+				(font
+					(size 1.27 1.27)
+				)
+			)
+		)
+		(property "MPN" ""
+			(at 71.12 116.84 0)
+			(hide yes)
+			(show_name no)
+			(do_not_autoplace no)
+			(effects
+				(font
+					(size 1.27 1.27)
+				)
+			)
+		)
+		(property "JLCPCB Part#" ""
+			(at 71.12 116.84 0)
+			(hide yes)

Commit message: Adding MPN to parts
Parts:
- C42: JLCPCB Part# (none) -> C2895275; MPN (none) -> RVT10UF16V67RV0012
- M1: JLCPCB Part# (none) -> C240840; MPN (none) -> 470531000
- R38: footprint Resistor_SMD:R_0402_1005Metric -> Resistor_SMD:R_0603_1608Metric; JLCPCB Part# (none) -> C844135; MPN (none) -> CRCW06031K00JNEAC
Changed lines of the file:
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@@
+			)
+		)
+		(property "v" ""
+			(at 82.55 116.84 0)
+			(hide yes)
+			(show_name no)
+			(do_not_autoplace no)
+			(effects
+				(font
+					(size 1.27 1.27)
+				)
 			)
 		)
@@
 			)
 		)
-		(property "Footprint" "Resistor_SMD:R_0402_1005Metric"
+		(property "Footprint" "Resistor_SMD:R_0603_1608Metric"
 			(at 210.312 111.76 90)
 			(hide yes)
@@
 		)
 		(property "MP" ""
+			(at 212.09 111.76 0)
+			(hide yes)
+			(show_name no)
+			(do_not_autoplace no)
+			(effects
+				(font
+					(size 1.27 1.27)
+				)
+			)
+		)
+		(property "MPN" "CRCW06031K00JNEAC"
+			(at 212.09 111.76 0)
+			(hide yes)
+			(show_name no)
+			(do_not_autoplace no)
+			(effects
+				(font
+					(size 1.27 1.27)
+				)
+			)
+		)
+		(property "JLCPCB Part#" "C844135"
+			(at 212.09 111.76 0)
+			(hide yes)
+			(show_name no)
+			(do_not_autoplace no)
+			(effects
+				(font
+					(size 1.27 1.27)
+				)
+			)
+		)
+		(property "v" ""
 			(at 212.09 111.76 0)
 			(hide yes)
@@
 			)
 		)
+		(property "v" ""
+			(at 147.32 100.33 0)
+			(hide yes)
+			(show_name no)
+			(do_not_autoplace no)
+			(effects
+				(font
+					(size 1.27 1.27)
+				)
+			)
+		)
 		(pin "14"
 		)
@@
 			)
 		)
+		(property "MPN" "470531000"
+			(at 222.25 120.65 0)
+			(hide yes)
+			(show_name no)
+			(do_not_autoplace no)
+			(effects
+				(font
+					(size 1.27 1.27)
+				)
+			)
+		)
+		(property "JLCPCB Part#" "C240840"
+			(at 222.25 120.65 0)
+			(hide yes)
+			(show_name no)
+			(do_not_autoplace no)
+			(effects
+				(font
+					(size 1.27 1.27)
+				)
+			)
+		)
+		(property "v" ""
+			(at 222.25 120.65 0)
+			(hide yes)
+			(show_name no)
+			(do_not_autoplace no)
+			(effects
+				(font
+					(size 1.27 1.27)
+				)
+			)
+		)
 		(pin "1"
 		)
@@
 			)
 		)
-		(property "MPN" ""
+		(property "MPN" "RVT10UF16V67RV0012"
 			(at 71.12 116.84 0)
 			(hide yes)
@@
 			)
 		)
-		(property "JLCPCB Part#" ""
+		(property "JLCPCB Part#" "C2895275"
 			(at 71.12 116.84 0)
 			(hide yes)
+			(show_name no)
+			(do_not_autoplace no)
+			(effects
+				(font
+					(size 1.27 1.27)
+				)
+			)
+		)
+		(property "v" ""
+			(at 71.12 116.84 0)
+			(hide yes)

Commit message: Replacing components
Parts:
- C42: footprint Capacitor_SMD:CP_Elec_4x4.5 -> Capacitor_SMD:C_0805_2012Metric; symbol Device:C_Polarized -> Device:C; JLCPCB Part# C2895275 -> C41893; MPN RVT10UF16V67RV0012 -> CL21A106MQFNNNE
- J14, M1: now left out of the parts list
Changed lines of the file:
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@@
 		(body_style 1)
 		(exclude_from_sim no)
-		(in_bom yes)
+		(in_bom no)
 		(on_board yes)
 		(in_pos_files yes)
@@
 		(body_style 1)
 		(exclude_from_sim no)
-		(in_bom yes)
+		(in_bom no)
 		(on_board yes)
 		(in_pos_files yes)
@@
 	)
 	(symbol
-		(lib_id "Device:C_Polarized")
+		(lib_id "Device:C")
 		(at 71.12 116.84 0)
 		(unit 1)
@@
 		(fields_autoplaced yes)
 		(property "Reference" "C42"
-			(at 74.93 114.6809 0)
+			(at 74.93 115.5699 0)
 			(show_name no)
 			(do_not_autoplace no)
@@
 		)
 		(property "Value" "10uF"
-			(at 74.93 117.2209 0)
+			(at 74.93 118.1099 0)
 			(show_name no)
 			(do_not_autoplace no)
@@
 			)
 		)
-		(property "Footprint" "Capacitor_SMD:CP_Elec_4x4.5"
+		(property "Footprint" "Capacitor_SMD:C_0805_2012Metric"
 			(at 72.0852 120.65 0)
 			(hide yes)
@@
 			)
 		)
-		(property "Description" "Polarized capacitor"
+		(property "Description" "Unpolarized capacitor"
 			(at 71.12 116.84 0)
 			(hide yes)
@@
 			)
 		)
-		(property "MPN" "RVT10UF16V67RV0012"
+		(property "MPN" "CL21A106MQFNNNE"
 			(at 71.12 116.84 0)
 			(hide yes)
@@
 			)
 		)
-		(property "JLCPCB Part#" "C2895275"
+		(property "JLCPCB Part#" "C41893"
 			(at 71.12 116.84 0)
 			(hide yes)

Commit message: Updating schematic
Parts:
- C42: JLCPCB Part # (none) -> C41893; JLCPCB Part# C41893 -> (none)
- C43: JLCPCB Part # (none) -> C307331; JLCPCB Part# C307331 -> (none)
- M1: JLCPCB Part # (none) -> C240840; JLCPCB Part# C240840 -> (none)
- R38: JLCPCB Part # (none) -> C844135; JLCPCB Part# C844135 -> (none)
Changed lines of the file:
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@@
-			)
-		)
-		(property "Sim.Device" ""
-			(at 82.55 116.84 0)
-			(hide yes)
-			(show_name no)
-			(do_not_autoplace no)
-			(effects
-				(font
-					(size 1.27 1.27)
-				)
-			)
-		)
-		(property "Sim.Type" ""
-			(at 82.55 116.84 0)
-			(hide yes)
-			(show_name no)
-			(do_not_autoplace no)
-			(effects
-				(font
-					(size 1.27 1.27)
-				)
 			)
 		)
@@
 			)
 		)
-		(property "JLCPCB Part#" "C307331"
+		(property "JLCPCB Part #" "C307331"
 			(at 82.55 116.84 0)
 			(hide yes)
@@
 			)
 		)
-		(property "v" ""
+		(property "MANUFACTURER" ""
+			(at 82.55 116.84 0)
+			(hide yes)
+			(show_name no)
+			(do_not_autoplace no)
+			(effects
+				(font
+					(size 1.27 1.27)
+				)
+			)
+		)
+		(property "MAXIMUM_PACKAGE_HEIGHT" ""
+			(at 82.55 116.84 0)
+			(hide yes)
+			(show_name no)
+			(do_not_autoplace no)
+			(effects
+				(font
+					(size 1.27 1.27)
+				)
+			)
+		)
+		(property "PARTREV" ""
 			(at 82.55 116.84 0)
 			(hide yes)
@@
 			)
 		)
-		(property "Sim.Device" ""
-			(at 212.09 111.76 0)
-			(hide yes)
-			(show_name no)
-			(do_not_autoplace no)
-			(effects
-				(font
-					(size 1.27 1.27)
-				)
-			)
-		)
-		(property "Sim.Type" ""
-			(at 212.09 111.76 0)
-			(hide yes)
-			(show_name no)
-			(do_not_autoplace no)
-			(effects
-				(font
-					(size 1.27 1.27)
-				)
-			)
-		)
 		(property "Author" ""
 			(at 212.09 111.76 0)
@@
 			)
 		)
-		(property "JLCPCB Part#" "C844135"
+		(property "JLCPCB Part #" "C844135"
 			(at 212.09 111.76 0)
 			(hide yes)
@@
 			)
 		)
-		(property "v" ""
+		(property "MANUFACTURER" ""
+			(at 212.09 111.76 0)
+			(hide yes)
+			(show_name no)
+			(do_not_autoplace no)
+			(effects
+				(font
+					(size 1.27 1.27)
+				)
+			)
+		)
+		(property "MAXIMUM_PACKAGE_HEIGHT" ""
+			(at 212.09 111.76 0)
+			(hide yes)
+			(show_name no)
+			(do_not_autoplace no)
+			(effects
+				(font
+					(size 1.27 1.27)
+				)
+			)
+		)
+		(property "PARTREV" ""
 			(at 212.09 111.76 0)
 			(hide yes)
@@
 			)
 		)
-		(property "v" ""
+		(property "MANUFACTURER" ""
+			(at 147.32 100.33 0)
+			(hide yes)
+			(show_name no)
+			(do_not_autoplace no)
+			(effects
+				(font
+					(size 1.27 1.27)
+				)
+			)
+		)
+		(property "MAXIMUM_PACKAGE_HEIGHT" ""
+			(at 147.32 100.33 0)
+			(hide yes)
+			(show_name no)
+			(do_not_autoplace no)
+			(effects
+				(font
+					(size 1.27 1.27)
+				)
+			)
+		)
+		(property "PARTREV" ""
 			(at 147.32 100.33 0)
 			(hide yes)
@@
 			)
 		)
-		(property "JLCPCB Part#" "C240840"
+		(property "JLCPCB Part #" "C240840"
 			(at 222.25 120.65 0)
 			(hide yes)
@@
 			)
 		)
-		(property "v" ""
+		(property "MANUFACTURER" ""
+			(at 222.25 120.65 0)
+			(hide yes)
+			(show_name no)
+			(do_not_autoplace no)
+			(effects
+				(font
+					(size 1.27 1.27)
+				)
+			)
+		)
+		(property "MAXIMUM_PACKAGE_HEIGHT" ""
+			(at 222.25 120.65 0)
+			(hide yes)
+			(show_name no)
+			(do_not_autoplace no)
+			(effects
+				(font
+					(size 1.27 1.27)
+				)
+			)
+		)
+		(property "PARTREV" ""
 			(at 222.25 120.65 0)
 			(hide yes)
@@
 			)
 		)
-		(property "Sim.Device" ""
-			(at 71.12 116.84 0)
-			(hide yes)
-			(show_name no)
-			(do_not_autoplace no)
-			(effects
-				(font
-					(size 1.27 1.27)
-				)
-			)
-		)
-		(property "Sim.Type" ""
-			(at 71.12 116.84 0)
-			(hide yes)
-			(show_name no)
-			(do_not_autoplace no)
-			(effects
-				(font
-					(size 1.27 1.27)
-				)
-			)
-		)
 		(property "Author" ""
 			(at 71.12 116.84 0)
@@
 			)
 		)
-		(property "JLCPCB Part#" "C41893"
+		(property "JLCPCB Part #" "C41893"
 			(at 71.12 116.84 0)
 			(hide yes)
@@
 			)
 		)
-		(property "v" ""
+		(property "MANUFACTURER" ""
 			(at 71.12 116.84 0)
 			(hide yes)
+			(show_name no)
+			(do_not_autoplace no)
+			(effects
+				(font
+					(size 1.27 1.27)
+				)
+			)
+		)
+		(property "MAXIMUM_PACKAGE_HEIGHT" ""
+			(at 71.12 116.84 0)
+			(hide yes)
+			(show_name no)
+			(do_not_autoplace no)
+			(effects
+				(font
+					(size 1.27 1.27)
+				)
+			)
+		)
+		(property "PARTREV" ""
+			(at 71.12 116.84 0)
+			(hide yes)
