File: hardware/stm32_mcu_core.kicad_sch (KiCad schematic)
At the start: 27 parts, among them J4 Conn_ST_STDC14, U6 SN74LVC1G126DBVR, U7 STM32G431KBTx, U8 SN74LVC1G125DBVR, U9 SN74AHCT1G125DBVR

Commit message: Adding external pullup to NRST
Parts:
- added R25: 10k, Resistor_SMD:R_0603_1608Metric, symbol Device:R
- renumbered R25 to R26, R26 to R27, R27 to R28, R28 to R29, R29 to R30, R30 to R31
Connections:
- net +3.3V: now also R25.1
- net NRST: now also R25.2

Commit message: Updating MPN and part number
Parts:
- D8, D9: JLCPCB Part# (none) -> C2890035; MPN (none) -> SK6805-EC15
- J4: JLCPCB Part# (none) -> C5563894; MFR FTSH-107-01-F-DV-K -> (none); MPN (none) -> FTSH-107-01-F-DV-K
- U6: JLCPCB Part# (none) -> C7834
- U7: JLCPCB Part# (none) -> C529357
- U8: JLCPCB Part# (none) -> C23654
- U9: JLCPCB Part# (none) -> C7484

Commit message: Updating BOM
Parts:
- C20, C21, C22, C23, C24, C27, C28, C29, C30: JLCPCB Part# (none) -> C307331; MPN (none) -> CL05B104KB54PNC
- C25: value 10µF -> 10uF; symbol Device:C -> Device:C_Polarized
- C26: value 1µF -> 1uF
Changed lines of the file:
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@@
 			)
 		)
+		(property "MPN" "CL05B104KB54PNC"
+			(at 38.1 181.61 0)
+			(hide yes)
+			(show_name no)
+			(do_not_autoplace no)
+			(effects
+				(font
+					(size 1.27 1.27)
+				)
+			)
+		)
+		(property "JLCPCB Part#" "C307331"
+			(at 38.1 181.61 0)
+			(hide yes)
+			(show_name no)
+			(do_not_autoplace no)
+			(effects
+				(font
+					(size 1.27 1.27)
+				)
+			)
+		)
 		(pin "2"
 		)
@@
 			)
 		)
+		(property "MPN" "CL05B104KB54PNC"
+			(at 22.86 181.61 0)
+			(hide yes)
+			(show_name no)
+			(do_not_autoplace no)
+			(effects
+				(font
+					(size 1.27 1.27)
+				)
+			)
+		)
+		(property "JLCPCB Part#" "C307331"
+			(at 22.86 181.61 0)
+			(hide yes)
+			(show_name no)
+			(do_not_autoplace no)
+			(effects
+				(font
+					(size 1.27 1.27)
+				)
+			)
+		)
 		(pin "2"
 		)
@@
 			)
 		)
+		(property "MPN" "CL05B104KB54PNC"
+			(at 115.57 181.61 0)
+			(hide yes)
+			(show_name no)
+			(do_not_autoplace no)
+			(effects
+				(font
+					(size 1.27 1.27)
+				)
+			)
+		)
+		(property "JLCPCB Part#" "C307331"
+			(at 115.57 181.61 0)
+			(hide yes)
+			(show_name no)
+			(do_not_autoplace no)
+			(effects
+				(font
+					(size 1.27 1.27)
+				)
+			)
+		)
 		(pin "2"
 		)
@@
 			)
 		)
+		(property "MPN" "CL05B104KB54PNC"
+			(at 132.08 181.61 0)
+			(hide yes)
+			(show_name no)
+			(do_not_autoplace no)
+			(effects
+				(font
+					(size 1.27 1.27)
+				)
+			)
+		)
+		(property "JLCPCB Part#" "C307331"
+			(at 132.08 181.61 0)
+			(hide yes)
+			(show_name no)
+			(do_not_autoplace no)
+			(effects
+				(font
+					(size 1.27 1.27)
+				)
+			)
+		)
 		(pin "2"
 		)
@@
 			)
 		)
+		(property "MPN" "CL05B104KB54PNC"
+			(at 73.66 181.61 0)
+			(hide yes)
+			(show_name no)
+			(do_not_autoplace no)
+			(effects
+				(font
+					(size 1.27 1.27)
+				)
+			)
+		)
+		(property "JLCPCB Part#" "C307331"
+			(at 73.66 181.61 0)
+			(hide yes)
+			(show_name no)
+			(do_not_autoplace no)
+			(effects
+				(font
+					(size 1.27 1.27)
+				)
+			)
+		)
 		(pin "2"
 		)
@@
 			)
 		)
+		(property "MPN" "CL05B104KB54PNC"
+			(at 162.56 181.61 0)
+			(hide yes)
+			(show_name no)
+			(do_not_autoplace no)
+			(effects
+				(font
+					(size 1.27 1.27)
+				)
+			)
+		)
+		(property "JLCPCB Part#" "C307331"
+			(at 162.56 181.61 0)
+			(hide yes)
+			(show_name no)
+			(do_not_autoplace no)
+			(effects
+				(font
+					(size 1.27 1.27)
+				)
+			)
+		)
 		(pin "2"
 		)
@@
 	)
 	(symbol
-		(lib_id "Device:C")
+		(lib_id "Device:C_Polarized")
 		(at 87.63 181.61 0)
 		(unit 1)
@@
 		(fields_autoplaced yes)
 		(property "Reference" "C25"
-			(at 91.44 180.3399 0)
+			(at 91.44 179.4509 0)
 			(show_name no)
 			(do_not_autoplace no)
@@
 			)
 		)
-		(property "Value" "10µF"
-			(at 91.44 182.8799 0)
+		(property "Value" "10uF"
+			(at 91.44 181.9909 0)
 			(show_name no)
 			(do_not_autoplace no)
@@
 			)
 		)
-		(property "Description" "Unpolarized capacitor"
+		(property "Description" "Polarized capacitor"
 			(at 87.63 181.61 0)
 			(hide yes)
@@
 			)
 		)
+		(property "MPN" ""
+			(at 87.63 181.61 0)
+			(hide yes)
+			(show_name no)
+			(do_not_autoplace no)
+			(effects
+				(font
+					(size 1.27 1.27)
+				)
+			)
+		)
+		(property "JLCPCB Part#" ""
+			(at 87.63 181.61 0)
+			(hide yes)
+			(show_name no)
+			(do_not_autoplace no)
+			(effects
+				(font
+					(size 1.27 1.27)
+				)
+			)
+		)
 		(pin "2"
 		)
@@
 			)
 		)
+		(property "MPN" "CL05B104KB54PNC"
+			(at 147.32 181.61 0)
+			(hide yes)
+			(show_name no)
+			(do_not_autoplace no)
+			(effects
+				(font
+					(size 1.27 1.27)
+				)
+			)
+		)
+		(property "JLCPCB Part#" "C307331"
+			(at 147.32 181.61 0)
+			(hide yes)
+			(show_name no)
+			(do_not_autoplace no)
+			(effects
+				(font
+					(size 1.27 1.27)
+				)
+			)
+		)
 		(pin "2"
 		)
@@
 			)
 		)
-		(property "Value" "1µF"
+		(property "Value" "1uF"
 			(at 107.95 182.8799 0)
 			(show_name no)
@@
 			)
 		)
+		(property "MPN" "CL05B104KB54PNC"
+			(at 135.89 72.39 0)
+			(hide yes)
+			(show_name no)
+			(do_not_autoplace no)
+			(effects
+				(font
+					(size 1.27 1.27)
+				)
+			)
+		)
+		(property "JLCPCB Part#" "C307331"
+			(at 135.89 72.39 0)
+			(hide yes)
+			(show_name no)
+			(do_not_autoplace no)
+			(effects
+				(font
+					(size 1.27 1.27)
+				)
+			)
+		)
 		(pin "2"
 		)
@@
 			(at 59.69 181.61 0)
 			(hide yes)
+			(show_name no)
+			(do_not_autoplace no)
+			(effects
+				(font
+					(size 1.27 1.27)
+				)
+			)
+		)
+		(property "MPN" "CL05B104KB54PNC"
+			(at 59.69 181.61 0)
+			(hide yes)
+			(show_name no)
+			(do_not_autoplace no)
+			(effects
+				(font
+					(size 1.27 1.27)
+				)
+			)
+		)
+		(property "JLCPCB Part#" "C307331"
+			(at 59.69 181.61 0)
+			(hide yes)

Commit message: Adding MPN to parts
Parts:
- C25: JLCPCB Part# (none) -> C2895275; MPN (none) -> RVT10UF16V67RV0012
- C26: JLCPCB Part# (none) -> C49326357; MPN (none) -> 0603X5R105K160NT
- D8: value SK6812_1 -> SK6812
- D9: value SK6812_2 -> SK6812
- FB1: value FerriteBead_Small -> FerriteBead; MPN (none) -> XRCB2012U201-2R5TF; Manufacturer (none) -> C41384131
- R25: footprint Resistor_SMD:R_0603_1608Metric -> Resistor_SMD:R_0402_1005Metric; JLCPCB Part# (none) -> C191984; MPN (none) -> CRCW040210K0JNED
- R26, R29: JLCPCB Part# (none) -> C191984; MPN (none) -> CRCW040210K0JNED
- R27, R28: JLCPCB Part# (none) -> C82865; MPN (none) -> CRCW0402100RFKED
- R30: footprint Resistor_SMD:R_0603_1608Metric -> Resistor_SMD:R_0402_1005Metric; MPN (none) -> CRCW040210K0JNED
- R31: footprint Resistor_SMD:R_0603_1608Metric -> Resistor_SMD:R_0402_1005Metric; JLCPCB Part# (none) -> C2906929; MPN (none) -> FRC0402J331 TS
- TP5, TP6: now left out of the parts list

Commit message: Replacing components
Parts:
- C25: footprint Capacitor_SMD:CP_Elec_4x4.5 -> Capacitor_SMD:C_0805_2012Metric; symbol Device:C_Polarized -> Device:C; JLCPCB Part# C2895275 -> C41893; MPN RVT10UF16V67RV0012 -> CL21A106MQFNNNE
- C26: JLCPCB Part# C49326357 -> C15849; MPN 0603X5R105K160NT -> CL10A105KB8NNNC
- FB1: JLCPCB Part# (none) -> C76819; MPN XRCB2012U201-2R5TF -> MPZ2012S331AT000; Manufacturer C41384131 -> (none)
- J4: now left out of the parts list
- R31: JLCPCB Part# C2906929 -> C25104; MPN FRC0402J331 TS -> 0402WGF3300TCE
Changed lines of the file:
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@@
 	)
 	(symbol
-		(lib_id "Device:C_Polarized")
+		(lib_id "Device:C")
 		(at 87.63 181.61 0)
 		(unit 1)
@@
 		(fields_autoplaced yes)
 		(property "Reference" "C25"
-			(at 91.44 179.4509 0)
+			(at 91.44 180.3399 0)
 			(show_name no)
 			(do_not_autoplace no)
@@
 		)
 		(property "Value" "10uF"
-			(at 91.44 181.9909 0)
+			(at 91.44 182.8799 0)
 			(show_name no)
 			(do_not_autoplace no)
@@
 			)
 		)
-		(property "Footprint" "Capacitor_SMD:CP_Elec_4x4.5"
+		(property "Footprint" "Capacitor_SMD:C_0805_2012Metric"
 			(at 88.5952 185.42 0)
 			(hide yes)
@@
 			)
 		)
-		(property "Description" "Polarized capacitor"
+		(property "Description" "Unpolarized capacitor"
 			(at 87.63 181.61 0)
 			(hide yes)
@@
 			)
 		)
-		(property "MPN" "RVT10UF16V67RV0012"
+		(property "MPN" "CL21A106MQFNNNE"
 			(at 87.63 181.61 0)
 			(hide yes)
@@
 			)
 		)
-		(property "JLCPCB Part#" "C2895275"
+		(property "JLCPCB Part#" "C41893"
 			(at 87.63 181.61 0)
 			(hide yes)
@@
 		(body_style 1)
 		(exclude_from_sim no)
-		(in_bom yes)
+		(in_bom no)
 		(on_board yes)
 		(in_pos_files yes)
@@
 			)
 		)
-		(property "MPN" "0603X5R105K160NT"
+		(property "MPN" "CL10A105KB8NNNC"
 			(at 104.14 181.61 0)
 			(hide yes)
@@
 			)
 		)
-		(property "JLCPCB Part#" "C49326357"
+		(property "JLCPCB Part#" "C15849"
 			(at 104.14 181.61 0)
 			(hide yes)
@@
 			)
 		)
-		(property "Manufacturer" "C41384131"
+		(property "Manufacturer" ""
 			(at 93.98 176.53 90)
 			(hide yes)
@@
 			)
 		)
-		(property "MPN" "XRCB2012U201-2R5TF"
+		(property "MPN" "MPZ2012S331AT000"
 			(at 93.98 176.53 0)
 			(hide yes)
@@
 			)
 		)
-		(property "JLCPCB Part#" ""
+		(property "JLCPCB Part#" "C76819"
 			(at 93.98 176.53 0)
 			(hide yes)
@@
 			)
 		)
-		(property "v" ""
-			(at 173.99 86.36 0)
-			(hide yes)
-			(show_name no)
-			(do_not_autoplace no)
-			(effects
-				(font
-					(size 1.27 1.27)
-				)
-			)
-		)
 		(pin "19"
 		)
@@
 			)
 		)
-		(property "MPN" "FRC0402J331 TS"
+		(property "MPN" "0402WGF3300TCE"
 			(at 251.46 113.03 0)
 			(hide yes)
@@
 			)
 		)
-		(property "JLCPCB Part#" "C2906929"
+		(property "JLCPCB Part#" "C25104"
 			(at 251.46 113.03 0)
 			(hide yes)

Commit message: Updating schematic
Parts:
- C20, C21, C22, C23, C24, C27, C28, C29, C30: JLCPCB Part # (none) -> C307331; JLCPCB Part# C307331 -> (none)
- C25: JLCPCB Part # (none) -> C41893; JLCPCB Part# C41893 -> (none)
- C26: JLCPCB Part # (none) -> C15849; JLCPCB Part# C15849 -> (none)
- D8, D9: JLCPCB Part # (none) -> C2890035; JLCPCB Part# C2890035 -> (none)
- FB1: JLCPCB Part # (none) -> C76819; JLCPCB Part# C76819 -> (none)
- J4: JLCPCB Part # (none) -> C5563894; JLCPCB Part# C5563894 -> (none)
- R25, R26, R29: JLCPCB Part # (none) -> C191984; JLCPCB Part# C191984 -> (none)
- R27, R28: JLCPCB Part # (none) -> C82865; JLCPCB Part# C82865 -> (none)
- R31: JLCPCB Part # (none) -> C25104; JLCPCB Part# C25104 -> (none)
- U6: JLCPCB Part # (none) -> C7834; JLCPCB Part# C7834 -> (none)
- U7: JLCPCB Part # (none) -> C529357; JLCPCB Part# C529357 -> (none)
- U8: JLCPCB Part # (none) -> C23654; JLCPCB Part# C23654 -> (none)
- U9: JLCPCB Part # (none) -> C7484; JLCPCB Part# C7484 -> (none)
