File: hardware/stm32_mcu_core.kicad_sch (KiCad schematic)
At the start: 28 parts, among them J4 Conn_ST_STDC14, U6 SN74LVC1G126DBVR, U7 STM32G431KBTx, U8 SN74LVC1G125DBVR, U9 SN74AHCT1G125DBVR

Commit message: schematic update
Parts:
- removed D8: SK6812, LED_SMD:LED_SK6812_EC15_1.5x1.5mm, symbol LED:SK6812
- removed J4: Conn_ST_STDC14, Chromapi_FP:SAMTEC_FTSH-107-01-L-DV-K-A, symbol Connector:Conn_ST_STDC14
- added J4: RGB LED Ring, Connector_JST:JST_XH_B3B-XH-A_1x03_P2.50mm_Vertical, symbol Connector_Generic:Conn_01x03
- D9: now not fitted
Connections:
- net +5V: now also J4.1 (Pin_1)
- net GND: now also J4.3 (Pin_3)
- net BOOT: now reaches R30.1, U7.31 (PB8)
- net at R31.1: now also J4.2 (Pin_2)
- no-connect marks 7 -> 3
Other:
- moved on the sheet: R31, U9
