File: hardware/stm32_mcu_core.kicad_sch (KiCad schematic)
At the start: 26 parts, among them J4 RGB LED Ring, U6 SN74LVC1G126DBVR, U7 STM32G431KBTx, U8 SN74AHCT1G125DBVR, U9 SN74LVC1G125DBVR

Commit message: bom optimisation for pcba
Parts:
- C25: JLCPCB Part # C41893 -> C15850; MPN CL21A106MQFNNNE -> CL21A106KAYNNNE
- R23, R24, R28: JLCPCB Part # C191984 -> C25744; MPN CRCW040210K0JNED -> 0402WGF1002TCE
- R25, R27: JLCPCB Part # C82865 -> C11702; MPN CRCW0402100RFKED -> 0402WGF1001TCE
- R29: JLCPCB Part # C60490 -> C25744; MPN RC0402FR-0710KL -> 0402WGF1002TCE
- U6: FT Rotation Offset (none) -> 180
- U9: FT Rotation Offset (none) -> -90
Changed lines of the file:
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@@
 			)
 		)
-		(property "MPN" "CRCW0402100RFKED"
+		(property "MPN" "0402WGF1001TCE"
 			(at 100.33 97.79 0)
 			(hide yes)
@@
 			)
 		)
-		(property "JLCPCB Part #" "C82865"
+		(property "JLCPCB Part #" "C11702"
 			(at 100.33 97.79 0)
 			(hide yes)
@@
 			)
 		)
-		(property "MPN" "CRCW0402100RFKED"
+		(property "MPN" "0402WGF1001TCE"
 			(at 74.93 74.93 0)
 			(hide yes)
@@
 			)
 		)
-		(property "JLCPCB Part #" "C82865"
+		(property "JLCPCB Part #" "C11702"
 			(at 74.93 74.93 0)
 			(hide yes)
@@
 			)
 		)
-		(property "MPN" "RC0402FR-0710KL"
+		(property "MPN" "0402WGF1002TCE"
 			(at 152.4 104.14 0)
 			(hide yes)
@@
 			)
 		)
-		(property "JLCPCB Part #" "C60490"
+		(property "JLCPCB Part #" "C25744"
 			(at 152.4 104.14 0)
 			(hide yes)
@@
 			)
 		)
-		(property "MPN" "CRCW040210K0JNED"
+		(property "MPN" "0402WGF1002TCE"
 			(at 58.42 100.33 0)
 			(hide yes)
@@
 			)
 		)
-		(property "JLCPCB Part #" "C191984"
+		(property "JLCPCB Part #" "C25744"
 			(at 58.42 100.33 0)
 			(hide yes)
@@
 			)
 		)
+		(property "FT Rotation Offset" "-90"
+			(at 81.28 101.6 0)
+			(hide yes)
+			(show_name no)
+			(do_not_autoplace no)
+			(effects
+				(font
+					(size 1.27 1.27)
+				)
+			)
+		)
 		(pin "1"
 		)
@@
 			)
 		)
-		(property "MPN" "CRCW040210K0JNED"
+		(property "MPN" "0402WGF1002TCE"
 			(at 142.24 59.69 0)
 			(hide yes)
@@
 			)
 		)
-		(property "JLCPCB Part #" "C191984"
+		(property "JLCPCB Part #" "C25744"
 			(at 142.24 59.69 0)
 			(hide yes)
@@
 			)
 		)
-		(property "MPN" "CL21A106MQFNNNE"
+		(property "MPN" "CL21A106KAYNNNE"
 			(at 93.98 180.34 0)
 			(hide yes)
@@
 			)
 		)
-		(property "JLCPCB Part #" "C41893"
+		(property "JLCPCB Part #" "C15850"
 			(at 93.98 180.34 0)
 			(hide yes)
@@
 			)
 		)
+		(property "FT Rotation Offset" "180"
+			(at 45.72 81.28 0)
+			(hide yes)
+			(show_name no)
+			(do_not_autoplace no)
+			(effects
+				(font
+					(size 1.27 1.27)
+				)
+			)
+		)
 		(pin "1"
 		)
@@
 			)
 		)
-		(property "MPN" "CRCW040210K0JNED"
+		(property "MPN" "0402WGF1002TCE"
 			(at 85.09 69.85 0)
 			(hide yes)
@@
 			)
 		)
-		(property "JLCPCB Part #" "C191984"
+		(property "JLCPCB Part #" "C25744"
 			(at 85.09 69.85 0)
 			(hide yes)
